Commit message: housekeeping?

File: urdf/turtlebot_urdf.xacro (robot description, xacro)
@@ -8,5 +8,5 @@
   <inertial>
     <origin xyz="-0.011892043852621992 -0.0005619831717906164 0.09178014322322671" rpy="0 0 0"/>
-    <mass value="3.029194688421112"/>
+    <mass value="5.029194688421112"/>
     <inertia ixx="0.005252" iyy="0.008834" izz="0.00825" ixy="-8e-06" iyz="2e-06" ixz="-0.000662"/>
   </inertial>

Commit message: wheelTest?

File: urdf/turtlebot_urdf.xacro (robot description, xacro)
@@ -28,11 +28,11 @@
   <inertial>
     <origin xyz="0.06888830561351354 -0.023235974830111583 0.023835792094402966" rpy="0 0 0"/>
-    <mass value="0.03203126833465021"/>
-    <inertia ixx="1.4e-05" iyy="2.4e-05" izz="1.4e-05" ixy="-0.0" iyz="0.0" ixz="0.0"/>
+    <mass value="0.16015634167325105"/>
+    <inertia ixx="0.000401" iyy="0.000401" izz="0.00007207" ixy="0.0" iyz="0.0" ixz="0.0"/>
   </inertial>
   <visual>
     <origin xyz="0.06353 0.0615 -0.034204" rpy="0 0 0"/>
     <geometry>
-      <mesh filename="file://$(find turtlebot)/meshes/wheel_2.stl" scale="0.001 0.001 0.001"/>
+      <mesh filename="file://$(find turtlebot)/meshes/wheel_2.stl" scale="0.001 0.001 0.05"/>
     </geometry>
     <material name="blue"/>
@@ -41,6 +41,20 @@
     <origin xyz="0.06353 0.0615 -0.034204" rpy="0 0 0"/>
     <geometry>
-      <mesh filename="file://$(find turtlebot)/meshes/wheel_2.stl" scale="0.001 0.001 0.001"/>
+      <mesh filename="file://$(find turtlebot)/meshes/wheel_2.stl" scale="0.001 0.001 0.05"/>
     </geometry>
+    <surface>
+      <friction>
+        <ode>
+          <mu>1.0</mu>
+          <mu2>1.0</mu2>
+        </ode>
+      </friction>
+      <contact>
+        <ode>
+          <kp>100000</kp>
+          <kd>1</kd>
+        </ode>
+      </contact>
+    </surface>
   </collision>
 </link>
@@ -48,11 +62,11 @@
   <inertial>
     <origin xyz="3.056135131906945e-07 0.01829722739215528 -1.1901500950733945e-07" rpy="0 0 0"/>
-    <mass value="0.03203126833465021"/>
-    <inertia ixx="1.4e-05" iyy="2.4e-05" izz="1.4e-05" ixy="0.0" iyz="0.0" ixz="-0.0"/>
+    <mass value="0.16015634167325105"/>
+    <inertia ixx="0.000401" iyy="0.000401" izz="0.00007207" ixy="0.0" iyz="0.0" ixz="0.0"/>
   </inertial>
   <visual>
     <origin xyz="0.06353 -0.065361 -0.034204" rpy="0 0 0"/>
     <geometry>
-      <mesh filename="file://$(find turtlebot)/meshes/wheel_1.stl" scale="0.001 0.001 0.001"/>
+      <mesh filename="file://$(find turtlebot)/meshes/wheel_1.stl" scale="0.001 0.001 0.05"/>
     </geometry>
     <material name="blue"/>
@@ -61,6 +75,20 @@
     <origin xyz="0.06353 -0.065361 -0.034204" rpy="0 0 0"/>
     <geometry>
-      <mesh filename="file://$(find turtlebot)/meshes/wheel_1.stl" scale="0.001 0.001 0.001"/>
+      <mesh filename="file://$(find turtlebot)/meshes/wheel_1.stl" scale="0.001 0.001 0.05"/>
     </geometry>
+    <surface>
+      <friction>
+        <ode>
+          <mu>1.0</mu>
+          <mu2>1.0</mu2>
+        </ode>
+      </friction>
+      <contact>
+        <ode>
+          <kp>100000</kp>
+          <kd>1</kd>
+        </ode>
+      </contact>
+    </surface>
   </collision>
 </link>

Commit message: backPropogate

File: urdf/turtlebot_urdf.xacro (robot description, xacro)
@@ -28,11 +28,11 @@
   <inertial>
     <origin xyz="0.06888830561351354 -0.023235974830111583 0.023835792094402966" rpy="0 0 0"/>
-    <mass value="0.16015634167325105"/>
-    <inertia ixx="0.000401" iyy="0.000401" izz="0.00007207" ixy="0.0" iyz="0.0" ixz="0.0"/>
+    <mass value="0.03203126833465021"/>
+    <inertia ixx="1.4e-05" iyy="2.4e-05" izz="1.4e-05" ixy="-0.0" iyz="0.0" ixz="0.0"/>
   </inertial>
   <visual>
     <origin xyz="0.06353 0.0615 -0.034204" rpy="0 0 0"/>
     <geometry>
-      <mesh filename="file://$(find turtlebot)/meshes/wheel_2.stl" scale="0.001 0.001 0.05"/>
+      <mesh filename="file://$(find turtlebot)/meshes/wheel_2.stl" scale="0.001 0.001 0.001"/>
     </geometry>
     <material name="blue"/>
@@ -41,5 +41,5 @@
     <origin xyz="0.06353 0.0615 -0.034204" rpy="0 0 0"/>
     <geometry>
-      <mesh filename="file://$(find turtlebot)/meshes/wheel_2.stl" scale="0.001 0.001 0.05"/>
+      <mesh filename="file://$(find turtlebot)/meshes/wheel_2.stl" scale="0.001 0.001 0.001"/>
     </geometry>
   </collision>
@@ -48,11 +48,11 @@
   <inertial>
     <origin xyz="3.056135131906945e-07 0.01829722739215528 -1.1901500950733945e-07" rpy="0 0 0"/>
-    <mass value="0.16015634167325105"/>
-    <inertia ixx="0.000401" iyy="0.000401" izz="0.00007207" ixy="0.0" iyz="0.0" ixz="0.0"/>
+    <mass value="0.03203126833465021"/>
+    <inertia ixx="1.4e-05" iyy="2.4e-05" izz="1.4e-05" ixy="0.0" iyz="0.0" ixz="-0.0"/>
   </inertial>
   <visual>
     <origin xyz="0.06353 -0.065361 -0.034204" rpy="0 0 0"/>
     <geometry>
-      <mesh filename="file://$(find turtlebot)/meshes/wheel_1.stl" scale="0.001 0.001 0.05"/>
+      <mesh filename="file://$(find turtlebot)/meshes/wheel_1.stl" scale="0.001 0.001 0.001"/>
     </geometry>
     <material name="blue"/>
@@ -61,5 +61,5 @@
     <origin xyz="0.06353 -0.065361 -0.034204" rpy="0 0 0"/>
     <geometry>
-      <mesh filename="file://$(find turtlebot)/meshes/wheel_1.stl" scale="0.001 0.001 0.05"/>
+      <mesh filename="file://$(find turtlebot)/meshes/wheel_1.stl" scale="0.001 0.001 0.001"/>
     </geometry>
   </collision>

Commit message: inertias

File: urdf/turtlebot_urdf.xacro (robot description, xacro)
@@ -28,6 +28,8 @@
   <inertial>
     <origin xyz="0.06888830561351354 -0.023235974830111583 0.023835792094402966" rpy="0 0 0"/>
-    <mass value="0.03203126833465021"/>
-    <inertia ixx="1.4e-05" iyy="2.4e-05" izz="1.4e-05" ixy="-0.0" iyz="0.0" ixz="0.0"/>
+    <mass value="0.05"/>
+   <inertia ixx="${(2/5) * 0.05 * (0.033*0.033)}" ixy="0.0" ixz="0.0"
+                    iyy="${(2/5) * 0.05 * (0.033*0.033)}" iyz="0.0"
+                    izz="${(2/5) * 0.05 * (0.033s*0.033)}" />
   </inertial>
   <visual>
@@ -48,6 +50,8 @@
   <inertial>
     <origin xyz="3.056135131906945e-07 0.01829722739215528 -1.1901500950733945e-07" rpy="0 0 0"/>
-    <mass value="0.03203126833465021"/>
-    <inertia ixx="1.4e-05" iyy="2.4e-05" izz="1.4e-05" ixy="0.0" iyz="0.0" ixz="-0.0"/>
+    <mass value="0.05"/>
+     <inertia ixx="${(2/5) * 0.05 * (0.033*0.033)}" ixy="0.0" ixz="0.0"
+                    iyy="${(2/5) * 0.05 * (0.033*0.033)}" iyz="0.0"
+                    izz="${(2/5) * 0.05 * (0.033s*0.033)}" />
   </inertial>
   <visual>

Commit message: inertia fix

File: urdf/turtlebot_urdf.xacro (robot description, xacro)
@@ -29,7 +29,7 @@
     <origin xyz="0.06888830561351354 -0.023235974830111583 0.023835792094402966" rpy="0 0 0"/>
     <mass value="0.05"/>
-   <inertia ixx="${(2/5) * 0.05 * (0.033*0.033)}" ixy="0.0" ixz="0.0"
-                    iyy="${(2/5) * 0.05 * (0.033*0.033)}" iyz="0.0"
-                    izz="${(2/5) * 0.05 * (0.033*0.033)}" />
+   <inertia ixx="${(1/12) * 0.05 * (3*0.033*0.033 + 0.026*0.026)}" ixy="0.0" ixz="0.0"
+                    iyy="${(1/12) * 0.05 * (3*0.033*0.033 + 0.026*0.026)}" iyz="0.0"
+                    izz="${(1/12) * 0.05 * (0.033*0.033)}" />
   </inertial>
   <visual>
@@ -51,7 +51,7 @@
     <origin xyz="3.056135131906945e-07 0.01829722739215528 -1.1901500950733945e-07" rpy="0 0 0"/>
     <mass value="0.05"/>
-     <inertia ixx="${(2/5) * 0.05 * (0.033*0.033)}" ixy="0.0" ixz="0.0"
-                    iyy="${(2/5) * 0.05 * (0.033*0.033)}" iyz="0.0"
-                    izz="${(2/5) * 0.05 * (0.033*0.033)}" />
+      <inertia ixx="${(1/12) * 0.05 * (3*0.033*0.033 + 0.026*0.026)}" ixy="0.0" ixz="0.0"
+                    iyy="${(1/12) * 0.05 * (3*0.033*0.033 + 0.026*0.026)}" iyz="0.0"
+                    izz="${(1/12) * 0.05 * (0.033*0.033)}" />
   </inertial>
   <visual>
