Commit message: encoder tic fix

File: description/lidar.xacro (robot description, xacro)
@@ -4,5 +4,5 @@
         <parent link="chassis"/>
         <child link="laser_frame"/>
-        <origin xyz="${2*chassis_length/3} 0 ${chassis_height+0.02}" rpy="0 0 0"/>
+        <origin xyz="${2*chassis_length/3} 0 ${chassis_height+0.02}" rpy="0 0 ${pi/2}"/>
     </joint>
     <link name="laser_frame">

File: description/ros2_control.xacro (robot description, xacro)
@@ -11,5 +11,5 @@
                 <param name="baud_rate">115200</param>
                 <param name="timeout">1000</param>
-                <param name="enc_counts_per_rev">660</param>
+                <param name="enc_counts_per_rev">410</param>
             </hardware>
             <joint name="left_wheel_joint">
